File: boards/dashboard_v1/controller.sch (EAGLE design)
At the start: 20 parts, among them J1 ARM_MINI_JTAG-TH, U1 LPC1114FN28, U3 24LC64P, U5 MCP2025DIL8, X1 2X2-A

Commit message: Part number fixes
Parts:
- C3, C4: PARTNO C1608X7R1H104M080AA -> FK28X7R1H104K
Changed lines of the file:
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@@
 </part>
 <part name="C3" library="custom" deviceset="C-EU" device="050-024X044" value="0u1">
-<attribute name="PARTNO" value="C1608X7R1H104M080AA"/>
+<attribute name="PARTNO" value="FK28X7R1H104K"/>
 </part>
 <part name="GND2" library="custom" deviceset="GND" device=""/>
@@
 </part>
 <part name="C4" library="custom" deviceset="C-EU" device="050-024X044" value="0u1">
-<attribute name="PARTNO" value="C1608X7R1H104M080AA"/>
+<attribute name="PARTNO" value="FK28X7R1H104K"/>
 </part>
 <part name="GND5" library="custom" deviceset="GND" device=""/>
